File: Hardware/SDMD/SDMD.kicad_pcb (KiCad board)
At the start: 2 copper layers, 25.4 x 25.7 mm, 19 parts, among them J1 Power, J2 Servo, J3 Servo, J4 AVR-ISP-6, J5 M1, J6 M2, U1 ATmega328-A, U2 AMS1117-5.0, U3 A4950E, U4 A4950E

Commit message: Rework
Parts:
- removed kibuzzard-64FD511C: G***, kibuzzard-64FD511C
- added kibuzzard-6781F98D: G***, kibuzzard-6781F98D, F.Cu at (131.8, 57.1)
- moved C1 0.38 mm to (133.2, 54.1)
- moved J1 0.19 mm to (139.4, 54.4)
Connections:
- J4 pad 1: /MOSI -> /MISO
- J4 pad 4: /MISO -> /MOSI
Routing:
- net /MISO: track 11.1 -> 14.3 mm, vias 2 -> 4
- net /MOSI: track 16.4 -> 14.0 mm
Other:
- board text added: "TX"
- board text added: "VIN"
