File: Hardware/SDMD/SDMD.kicad_sch (KiCad schematic)
At the start: 18 parts, among them J1 Power, J2 Servo, J3 Servo, J4 AVR-ISP-6, J5 M1, J6 M2, U1 ATmega328-A, U2 AMS1117-5.0, U3 A4950E, U4 A4950E

Commit message: Rework
Connections:
- net MISO: now also J4.1 (MISO); no longer J4.4 (MOSI)
- net MOSI: now also J4.4 (MOSI); no longer J4.1 (MISO)
