File: Hardware/Receiver USB/Receiver USB.kicad_sch (KiCad schematic)
At the start: 0 parts

Commit message: new USB receiver based on the Pro Micro
Parts:
- added C1: C, Capacitor_SMD:C_0805_2012Metric, symbol Device:C
- added J1: Conn_01x03_Socket, Connector_PinHeader_2.54mm:PinHeader_1x03_P2.54mm_Vertical, symbol Connector:Conn_01x03_Socket
- added J2: ~, user:SPARKFUN_PRT-14417, symbol user:Qwiic
- added U1: Sparkfun_Pro_Micro, Arduino Modules:Sparkfun_Pro_Micro, symbol Arduino Modules:Sparkfun_Pro_Micro
- added U2: AMS1117-3.3, Package_TO_SOT_SMD:SOT-223-3_TabPin2, symbol Regulator_Linear:AMS1117-3.3
- added U3: NRF24L01_Breakout, RF_Module:nRF24L01_Breakout, symbol RF:NRF24L01_Breakout
Connections:
- new net: J1.1 (Pin_1), U1.6 (~D3)
- new net: J2.1 (TX), U1.1 (D1/TX)
- new net: J2.2 (RX), U1.2 (D0/RX)
- new net +3V3: C1.2, U2.2 (VO), U3.2 (VCC)
- new net +5V: J1.2 (Pin_2), J2.3 (VCC), U2.3 (VI)
- new net CE: U1.12 (~D9/A9), U3.3 (CE)
- new net GND: C1.1, J1.3 (Pin_3), J2.4 (GND), J2.S1 (MNT), J2.S2 (MNT), U1.23 (GND), U1.3 (GND), U1.4 (GND), U2.1 (GND), U3.1 (GND)
- new net PICO: U1.15 (D14), U3.7 (MISO)
- new net POCI: U1.14 (D16), U3.6 (MOSI)
- new net SCK: U1.16 (D15), U3.5 (SCK)
- new net ~{CSN}: U1.13 (~D10/A10), U3.4 (~{CSN})
- no-connect marks 0 -> 16
