File: Hardware/Receiver USB/Receiver USB.kicad_pcb (KiCad board)
At the start: 2 copper layers, 19.3 x 33.7 mm, 6 parts, among them J1 Conn_01x03_Socket, U1 Sparkfun_Pro_Micro, U2 AMS1117-3.3, U3 NRF24L01_Breakout

Commit message: I ordered the receiver, tx, and sdmd kllip boards so I hope they work
Parts:
- added kibuzzard-67BFB299: G***, kibuzzard-67BFB299, F.Cu at (23.1, 22.7)
