File: Hardware/Generation 3 Transmitter/gen.kicad_pcb (KiCad board)
At the start: 2 copper layers, 99 x 48.5 mm, 23 parts, among them SW1 POWER, SW2 INVERT, U1 LEFT STICK, U2 RIGHT STICK, U3 ADS7830, U4 DISPLAY, U5 XIAO, U6 NRF24L01_Breakout

Commit message: Redoing the SDMD Kllip in an intelligent way, changing some receiver things, and designing a transmitter board
Parts:
- removed D1: WHITE, Connector_PinHeader_2.54mm:PinHeader_1x02_P2.54mm_Vertical
- removed D2: RED, Connector_PinHeader_2.54mm:PinHeader_1x02_P2.54mm_Vertical
- removed R2, R3: 10k, Resistor_SMD:R_0805_2012Metric
- removed R5: 220k, Resistor_SMD:R_0805_2012Metric
- C1, C3: value 10 -> 0.1; moved to F.Cu
- R1: value 1k -> 10k
- R8, R9, U3: moved to F.Cu
- moved U1 174.7 mm to (26.6, 27.5), turned to -90 degrees
- moved C3 163.7 mm to (50.0, 64.0)
- moved SW1 159.9 mm to (74.5, 16.5)
- moved SW2 159.4 mm to (79.0, 16.5)
- moved R1 157.3 mm to (81.4, 46.8), turned to -90 degrees
- moved U5 154.3 mm to (63.6, 60.6)
- moved U4 153.0 mm to (60.0, 16.5)
- moved U2 150.0 mm to (100.6, 27.5), turned to 90 degrees
- moved R7 145.2 mm to (65.3, 60.9), turned to 0 degrees
- moved R6 142.2 mm to (68.4, 58.0), turned to 180 degrees
- moved C1 139.6 mm to (54.5, 40.5), turned to -90 degrees
- moved U3 138.6 mm to (79.5, 53.6), turned to -90 degrees
- moved RV1 135.5 mm to (53.0, 18.0), turned to 0 degrees
- moved C2 133.8 mm to (80.5, 60.0), turned to 180 degrees
- moved U6 129.6 mm to (57.9, 47.3), turned to 90 degrees
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Connections:
- R1 pad 2: Net-(D1-K) -> Net-(SW2-A)
- SW2 pad 1: Net-(D1-A) -> Net-(SW2-A)
- U3 pad 2: Net-(D1-A) -> Net-(SW2-A)
- U5 pad 3: Net-(D2-A) -> unconnected-(U5-D2-Pad3)
Routing:
- net +3V3: track 186.1 -> 38.8 mm
- net /RY: track 15.4 -> 62.7 mm, vias 1 -> 0
- net Net-(SW1-A): track 52.1 -> 99.0 mm, vias 5 -> 3
- net Net-(D2-A): track 42.2 -> 0.00 mm
- net /LX: track 48.1 -> 90.2 mm, vias 2 -> 0
- net Net-(BT1--): track 16.9 -> 57.9 mm, vias 1 -> 0
- net Net-(U5-D0): track 6.16 -> 46.7 mm, vias 1 -> 2
- net Net-(D1-A): track 38.4 -> 0.00 mm, vias 1 -> 0
- net /SDA: track 28.8 -> 66.0 mm
- net Net-(SW2-A): track 0.00 -> 35.9 mm
- net /RX: track 30.7 -> 66.7 mm, vias 1 -> 0
- net Net-(U5-D6): track 53.5 -> 19.9 mm, vias 1 -> 0
- net /SCL: track 31.6 -> 64.3 mm, vias 2 -> 1
- net Net-(U5-D8): track 39.5 -> 12.4 mm
- net Net-(U5-D9): track 39.7 -> 17.2 mm
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- added copper zone on F.Cu, net +3V3
- added copper zone on B.Cu, net GND
- removed copper zone on F.Cu, net GND
Other:
- board size 99 x 48.5 mm -> 101 x 59.5 mm
