File: Hardware/SDMD Kllip 2/SDMD.kicad_pcb (KiCad board)
At the start: 2 copper layers, 25.4 x 25.7 mm, 19 parts, among them J1 Power, J2 Servo, J3 Servo, J4 AVR-ISP-6, J5 M1, J6 M2, U1 ATmega328-A, U2 AMS1117-5.0, U3 A4950E, U4 A4950E

Commit message: I ordered the receiver, tx, and sdmd kllip boards so I hope they work
Parts:
- removed J3: Servo, Connector_PinHeader_2.54mm:PinHeader_1x01_P2.54mm_Vertical
- added D1: LED, LED_SMD:LED_0805_2012Metric, F.Cu at (152.2, 52.6)
- added R4: 220, Resistor_SMD:R_0805_2012Metric, F.Cu at (152.1, 54.7)
- J2: value Servo -> Kllip; footprint Connector_PinHeader_2.54mm:PinHeader_1x03_P2.54mm_Vertical -> user:SPARKFUN_PRT-14417; moved to B.Cu
- J4: footprint Connector_PinHeader_2.54mm:PinHeader_2x03_P2.54mm_Vertical -> Connector_PinSocket_2.54mm:PinSocket_2x03_P2.54mm_Vertical; moved to B.Cu
- moved J2 1.75 mm to (132.3, 35.1), turned to 0 degrees
- moved J4 0.05 mm to (143.5, 54.5), turned to -90 degrees
Connections:
- J2 pad 1: GND -> /TX
- J2 pad 2: +5V -> /RX
- J2 pad 3: /RX -> +5V
- U1 pad 12: Net-(J3-Pin_1) -> unconnected-(U1-PB0-Pad12)
Routing:
- net Net-(J3-Pin_1): track 31.7 -> 0.00 mm, vias 2 -> 0
- net /TX: track 0.00 -> 5.52 mm, vias 0 -> 1
- net /RX: track 3.72 -> 7.51 mm, vias 0 -> 1
- net GND: track 9.70 -> 12.5 mm, vias 4 -> 5
- net Net-(D1-A): track 0.00 -> 2.15 mm
- net +5V: vias 6 -> 7
Other:
- board text removed: "TX"
