File: Hardware/SDMD Kllip 2/SDMD.kicad_sch (KiCad schematic)
At the start: 18 parts, among them J1 Power, J2 Servo, J3 Servo, J4 AVR-ISP-6, J5 M1, J6 M2, U1 ATmega328-A, U2 AMS1117-5.0, U3 A4950E, U4 A4950E

Commit message: I ordered the receiver, tx, and sdmd kllip boards so I hope they work
Parts:
- removed J2: Servo, Connector_PinHeader_2.54mm:PinHeader_1x03_P2.54mm_Vertical, symbol Connector:Conn_01x03_Pin
- removed J3: Servo, Connector_PinHeader_2.54mm:PinHeader_1x01_P2.54mm_Vertical, symbol Connector:Conn_01x01_Pin
- added D1: LED, LED_SMD:LED_0805_2012Metric, symbol Device:LED
- added J2: Kllip, user:SPARKFUN_PRT-14417, symbol user:Qwiic
- added R4: 220, Resistor_SMD:R_0805_2012Metric, symbol Device:R
- J4: footprint Connector_PinHeader_2.54mm:PinHeader_2x03_P2.54mm_Vertical -> Connector_PinSocket_2.54mm:PinSocket_2x03_P2.54mm_Vertical
Connections:
- net +5V: now also J2.3 (VCC), R4.1
- net GND: now also D1.1 (K), J2.4 (GND)
- net RX: now also J2.2 (RX)
- net TX: now also J2.1 (TX)
- new net: D1.2 (A), R4.2
- no-connect marks 0 -> 12
